File: beanzee-lcd-kbd/kicad/lcd-keypad/lcd-keypad.kicad_sch (KiCad schematic)
At the start: 29 parts, among them SW00 SW_Push_45deg, SW01 SW_Push_45deg, SW02 SW_Push_45deg, SW03 SW_Push_45deg, SW10 SW_Push_45deg, SW11 SW_Push_45deg, SW12 SW_Push_45deg, SW13 SW_Push_45deg, U1 74LS138, U1 74LS32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

Commit message: update schematics
Connections:
- net D2: no longer U2.7 (D2)
- net D3: no longer U2.8 (D3)
- net D4: no longer names the net of U3.9 (O0b)
- net D4: no longer U2.13 (D4)
- net D5: no longer names the net of U3.7 (O1b)
- net D5: no longer U2.14 (D5)
- net D6: no longer names the net of U3.5 (O2b)
- net D6: no longer U2.17 (D6)
- net D7: no longer names the net of U3.3 (O3b)
- net D7: no longer U2.18 (D7)
- no-connect marks 36 -> 46
Changed lines of the file:
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@@
   (no_connect (at 34.29 59.69))
   (no_connect (at 154.94 113.03))
+  (no_connect (at 180.34 118.11))
+  (no_connect (at 63.5 168.91))
   (no_connect (at 77.47 19.05))
   (no_connect (at 88.9 171.45))
+  (no_connect (at 63.5 176.53))
   (no_connect (at 119.38 46.99))
   (no_connect (at 77.47 44.45))
+  (no_connect (at 180.34 115.57))
   (no_connect (at 64.77 11.43))
   (no_connect (at 77.47 21.59))
+  (no_connect (at 63.5 181.61))
   (no_connect (at 77.47 16.51))
   (no_connect (at 88.9 181.61))
@@
   (no_connect (at 77.47 49.53))
   (no_connect (at 77.47 24.13))
+  (no_connect (at 63.5 171.45))
   (no_connect (at 77.47 54.61))
+  (no_connect (at 180.34 113.03))
+  (no_connect (at 63.5 179.07))
   (no_connect (at 119.38 44.45))
   (no_connect (at 119.38 49.53))
+  (no_connect (at 63.5 173.99))
   (no_connect (at 88.9 179.07))
   (no_connect (at 49.53 59.69))
@@
   (no_connect (at 88.9 176.53))
   (no_connect (at 54.61 11.43))
+  (no_connect (at 180.34 110.49))
   (no_connect (at 154.94 110.49))
   (no_connect (at 67.31 11.43))
@@
   (no_connect (at 52.07 11.43))
   (no_connect (at 62.23 11.43))
-  (bus_entry (at 46.99 168.91) (size 2.54 2.54)
-    (stroke (width 0) (type default))
-  )
   (bus_entry (at 3.81 207.01) (size 2.54 2.54)
     (stroke (width 0) (type default))
@@
     (stroke (width 0) (type default))
   )
-  (bus_entry (at 46.99 166.37) (size 2.54 2.54)
-    (stroke (width 0) (type default))
-  )
   (bus_entry (at 11.43 44.45) (size 2.54 2.54)
     (stroke (width 0) (type default))
@@
     (stroke (width 0) (type default))
   )
-  (wire (pts (xy 180.34 118.11) (xy 184.15 118.11))
-    (stroke (width 0) (type default))
-  )
   (wire (pts (xy 114.3 139.7) (xy 114.3 166.37))
     (stroke (width 0) (type default))
@@
     (stroke (width 0) (type default))
   )
-  (bus (pts (xy 46.99 166.37) (xy 46.99 168.91))
-    (stroke (width 0) (type default))
-  )
-  (wire (pts (xy 57.15 176.53) (xy 63.5 176.53))
-    (stroke (width 0) (type default))
-  )
   (wire (pts (xy 77.47 31.75) (xy 93.98 31.75))
     (stroke (width 0) (type default))
@@
     (stroke (width 0) (type default))
   )
-  (wire (pts (xy 57.15 181.61) (xy 63.5 181.61))
-    (stroke (width 0) (type default))
-  )
   (wire (pts (xy 186.69 17.78) (xy 172.72 17.78))
     (stroke (width 0) (type default))
@@
     (stroke (width 0) (type default))
   )
-  (wire (pts (xy 49.53 171.45) (xy 63.5 171.45))
-    (stroke (width 0) (type default))
-  )
   (wire (pts (xy 88.9 166.37) (xy 114.3 166.37))
     (stroke (width 0) (type default))
@@
     (stroke (width 0) (type default))
   )
-  (wire (pts (xy 49.53 168.91) (xy 63.5 168.91))
-    (stroke (width 0) (type default))
-  )
   (wire (pts (xy 186.69 49.53) (xy 186.69 68.58))
     (stroke (width 0) (type default))
@@
     (stroke (width 0) (type default))
   )
-  (wire (pts (xy 180.34 110.49) (xy 184.15 110.49))
-    (stroke (width 0) (type default))
-  )
   (wire (pts (xy 151.13 60.96) (xy 157.48 60.96))
     (stroke (width 0) (type default))
@@
     (stroke (width 0) (type default))
   )
-  (wire (pts (xy 57.15 179.07) (xy 63.5 179.07))
-    (stroke (width 0) (type default))
-  )
   (wire (pts (xy 96.52 100.33) (xy 111.76 100.33))
     (stroke (width 0) (type default))
@@
     (stroke (width 0) (type default))
   )
-  (wire (pts (xy 180.34 115.57) (xy 184.15 115.57))
-    (stroke (width 0) (type default))
-  )
   (wire (pts (xy 96.52 147.32) (xy 111.76 147.32))
     (stroke (width 0) (type default))
@@
     (stroke (width 0) (type default))
   )
-  (wire (pts (xy 180.34 113.03) (xy 184.15 113.03))
-    (stroke (width 0) (type default))
-  )
   (wire (pts (xy 90.17 29.21) (xy 77.47 29.21))
     (stroke (width 0) (type default))
@@
     (stroke (width 0) (type default))
   )
-  (bus (pts (xy 46.99 163.83) (xy 46.99 166.37))
-    (stroke (width 0) (type default))
-  )
   (wire (pts (xy 143.51 123.19) (xy 154.94 123.19))
     (stroke (width 0) (type default))
@@
   )
   (wire (pts (xy 167.64 90.17) (xy 167.64 92.71))
-    (stroke (width 0) (type default))
-  )
-  (wire (pts (xy 57.15 173.99) (xy 63.5 173.99))
     (stroke (width 0) (type default))
   )
@@
     (effects (font (size 1.27 1.27)) (justify left bottom))
   )
-  (label "D4" (at 184.15 110.49 0) (fields_autoplaced)
-    (effects (font (size 1.27 1.27)) (justify left bottom))
-  )
   (label "D3" (at 184.15 107.95 0) (fields_autoplaced)
     (effects (font (size 1.27 1.27)) (justify left bottom))
@@
     (effects (font (size 1.27 1.27)) (justify left bottom))
   )
-  (label "D3" (at 57.15 171.45 0) (fields_autoplaced)
-    (effects (font (size 1.27 1.27)) (justify left bottom))
-  )
   (label "D1" (at 57.15 166.37 0) (fields_autoplaced)
     (effects (font (size 1.27 1.27)) (justify left bottom))
   )
-  (label "D6" (at 57.15 179.07 0) (fields_autoplaced)
-    (effects (font (size 1.27 1.27)) (justify left bottom))
-  )
   (label "~{KB_RD}" (at 146.05 123.19 0) (fields_autoplaced)
     (effects (font (size 1.27 1.27)) (justify left bottom))
@@
     (effects (font (size 1.27 1.27)) (justify left bottom))
   )
-  (label "D5" (at 184.15 113.03 0) (fields_autoplaced)
-    (effects (font (size 1.27 1.27)) (justify left bottom))
-  )
-  (label "D7" (at 57.15 181.61 0) (fields_autoplaced)
-    (effects (font (size 1.27 1.27)) (justify left bottom))
-  )
   (label "D2" (at 184.15 105.41 0) (fields_autoplaced)
     (effects (font (size 1.27 1.27)) (justify left bottom))
   )
-  (label "D7" (at 184.15 118.11 0) (fields_autoplaced)
-    (effects (font (size 1.27 1.27)) (justify left bottom))
-  )
-  (label "D6" (at 184.15 115.57 0) (fields_autoplaced)
-    (effects (font (size 1.27 1.27)) (justify left bottom))
-  )
-  (label "D4" (at 57.15 173.99 0) (fields_autoplaced)
-    (effects (font (size 1.27 1.27)) (justify left bottom))
-  )
   (label "D1" (at 184.15 102.87 0) (fields_autoplaced)
     (effects (font (size 1.27 1.27)) (justify left bottom))
@@
     (effects (font (size 1.27 1.27)) (justify left bottom))
   )
-  (label "D2" (at 57.15 168.91 0) (fields_autoplaced)
-    (effects (font (size 1.27 1.27)) (justify left bottom))
-  )
   (label "D0" (at 184.15 100.33 0) (fields_autoplaced)
     (effects (font (size 1.27 1.27)) (justify left bottom))
@@
     (effects (font (size 1.27 1.27)) (justify left bottom))
   )
-  (label "D5" (at 57.15 176.53 0) (fields_autoplaced)
-    (effects (font (size 1.27 1.27)) (justify left bottom))
-  )
